File: pcb/fan.sch (KiCad schematic (older format))
At the start: 47 parts, among them J1 MJ-4PP-9, J2 Conn_01x01_Female, J3 Conn_01x01_Female, SW1 SW_PUSH-kbd, SW10 SW_PUSH-kbd, SW11 SW_PUSH-kbd, SW12 SW_PUSH-kbd, SW13 SW_PUSH-kbd, SW14 SW_PUSH-kbd, SW15 SW_PUSH-kbd, SW16 SW_PUSH-kbd, SW17 SW_PUSH-kbd, SW18 SW_PUSH-kbd, SW19 SW_PUSH-kbd, SW2 SW_PUSH-kbd, SW20 SW_PUSH-kbd, SW21 SW_PUSH-kbd, SW22 SW_PUSH-kbd, SW23 SW_PUSH-kbd, SW24 SW_PUSH-kbd, SW25 SW_PUSH-kbd, SW26 SW_PUSH-kbd, SW27 SW_PUSH-kbd, SW28 SW_PUSH-kbd, SW29 SW_PUSH-kbd, SW3 SW_PUSH-kbd, SW30 SW_PUSH-kbd, SW31 SW_PUSH-kbd, SW32 SW_PUSH-kbd, SW33 SW_PUSH-kbd, SW34 SW_PUSH-kbd, SW35 SW_PUSH-kbd, SW36 SW_PUSH-kbd, SW37 SW_PUSH-kbd, SW38 SW_PUSH-kbd, SW39 SW_PUSH-kbd, SW4 SW_PUSH-kbd, SW40 SW_PUSH-kbd, SW41 SW_PUSH, SW5 SW_PUSH-kbd, SW6 SW_PUSH-kbd, SW7 SW_PUSH-kbd, SW8 SW_PUSH-kbd, SW9 SW_PUSH-kbd, U1 BluePill_STM32F103C

Commit message: fan90専用のリポジトリにした
Parts:
- removed J1: MJ-4PP-9, kbd:MJ-4PP-9, symbol kbd:MJ-4PP-9
- removed J2, J3: Conn_01x01_Female, Connector_Pin:Pin_D1.0mm_L10.0mm, symbol Connector:Conn_01x01_Female
- removed R1, R2: 10K, keyboard_parts:R_1608_rev2, symbol Device:R
- removed SW1, SW11, SW12, SW13, SW14, SW16, SW17, SW18, SW19, SW2, SW20, SW21, SW22, SW23, SW24, SW25, SW26, SW27, SW28, SW29, SW3, SW30, SW31, SW32, SW33, SW34, SW35, SW36, SW37, SW38, SW39, SW4, SW40, SW6, SW7, SW8, SW9: SW_PUSH-kbd, kbd:CherryMX_MidHeight_Hotswap_edit, symbol New_Library:SW_PUSH-kbd
- removed SW10, SW15, SW5: SW_PUSH-kbd, kbd:ResetSW_with_diode, symbol New_Library:SW_PUSH-kbd
- removed U1: BluePill_STM32F103C, BluePill_breakouts:BluePill_STM32F103C_0.9_Double, symbol bluepill_breakouts:BluePill_STM32F103C
- added D1, D10, D11, D12, D13, D14, D15, D16, D17, D18, D19, D2, D20, D21, D22, D23, D24, D25, D26, D27, D28, D29, D3, D30, D31, D32, D33, D34, D35, D36, D37, D38, D39, D4, D40, D41, D42, D43, D44, D45, D46, D47, D48, D49, D5, D50, D51, D52, D53, D54, D55, D56, D57, D58, D59, D6, D60, D61, D62, D63, D64, D65, D66, D67, D68, D69, D7, D70, D71, D72, D73, D74, D75, D76, D77, D78, D79, D8, D80, D81, D82, D83, D84, D85, D86, D87, D88, D89, D9, D90: DIODE, kbd:D3_TH_SMD, symbol Device:D
- added J2: Pi, Connector_PinSocket_2.54mm:PinSocket_2x20_P2.54mm_Vertical, symbol fan-rescue:Connector_Generic_Conn_02x20_Odd_Even-Raspberry_Pi_Zero_W-cache
- added SW1, SW10, SW11, SW12, SW13, SW14, SW15, SW16, SW17, SW18, SW19, SW2, SW20, SW21, SW22, SW23, SW24, SW25, SW26, SW27, SW28, SW29, SW3, SW30, SW31, SW32, SW33, SW34, SW35, SW36, SW37, SW38, SW39, SW4, SW40, SW41, SW42, SW43, SW44, SW45, SW46, SW47, SW48, SW5, SW51, SW52, SW53, SW54, SW56, SW57, SW58, SW59, SW6, SW60, SW61, SW62, SW63, SW64, SW65, SW66, SW67, SW68, SW69, SW7, SW70, SW71, SW72, SW73, SW74, SW75, SW76, SW77, SW78, SW79, SW8, SW80, SW81, SW82, SW83, SW84, SW85, SW86, SW87, SW88, SW89, SW9, SW90: SW_PUSH, kbd:CherryMX_Hotswap, symbol fan-rescue:SW_PUSH-kbd
- added SW49, SW50, SW55, SW92: SW_PUSH, kbd:ResetSW, symbol fan-rescue:SW_PUSH-kbd
- added SW93: SW_SPDT, Button_Switch_THT:SW_Slide_1P2T_CK_OS102011MS2Q, symbol Switch:SW_SPDT
- added U1, U2: ProMicro, kbd:ProMicro_v3.6, symbol fan-rescue:ProMicro-kbd
- added U3, U4, U5, U6: 74HC595, kbd:SN74HC595_DIP-16_W7.62mm_Socket_2, symbol 74xx:74HC595
- renumbered SW41 to SW91
Connections:
- net labels added: OE, QHSER, QHSER', RCK, SCK, SCL, SER, col08, col09, col10, col11, col12, col13, col14, row05, software_reset
- net labels removed: Rx, Tx, data
- wire segments 104 -> 182
- no-connect marks 20 -> 58
Other:
- note removed: "A and B short circuit when using TRS plug"
- note removed: "insert ->"
- moved on the sheet: SW91
