File: pcb/fan.kicad_pcb (KiCad board)
At the start: 2 copper layers, 212.8 x 143.6 mm, 59 parts, among them J1 MJ-4PP-9, J2 Conn_01x01_Female, J3 Conn_01x01_Female, SW1 SW_PUSH-kbd, SW10 SW_PUSH-kbd, SW11 SW_PUSH-kbd, SW12 SW_PUSH-kbd, SW13 SW_PUSH-kbd, SW14 SW_PUSH-kbd, SW15 SW_PUSH-kbd, SW16 SW_PUSH-kbd, SW17 SW_PUSH-kbd, SW18 SW_PUSH-kbd, SW19 SW_PUSH-kbd, SW2 SW_PUSH-kbd, SW20 SW_PUSH-kbd, SW21 SW_PUSH-kbd, SW22 SW_PUSH-kbd, SW23 SW_PUSH-kbd, SW24 SW_PUSH-kbd, SW25 SW_PUSH-kbd, SW26 SW_PUSH-kbd, SW27 SW_PUSH-kbd, SW28 SW_PUSH-kbd, SW29 SW_PUSH-kbd, SW3 SW_PUSH-kbd, SW30 SW_PUSH-kbd, SW31 SW_PUSH-kbd, SW32 SW_PUSH-kbd, SW33 SW_PUSH-kbd, SW34 SW_PUSH-kbd, SW35 SW_PUSH-kbd, SW36 SW_PUSH-kbd, SW37 SW_PUSH-kbd, SW38 SW_PUSH-kbd, SW39 SW_PUSH-kbd, SW4 SW_PUSH-kbd, SW40 SW_PUSH-kbd, SW41 SW_PUSH, SW5 SW_PUSH-kbd, SW6 SW_PUSH-kbd, SW7 SW_PUSH-kbd, SW8 SW_PUSH-kbd, SW9 SW_PUSH-kbd, U1 BluePill_STM32F103C

Commit message: fan90専用のリポジトリにした
Parts:
- removed J1: MJ-4PP-9, kbd:MJ-4PP-9
- removed J3: Conn_01x01_Female, Connector_Pin:Pin_D1.0mm_L10.0mm
- removed R1, R2: 10K, keyboard_parts:R_1608_rev2
- removed Ref** (x12): Val**, kbd:HOLE
- added D1: DIODE, kbd:D3_TH_SMD, B.Cu at (53.8, 62.8)
- added D10: DIODE, kbd:D3_TH_SMD, B.Cu at (63.8, 118.1)
- added D11: DIODE, kbd:D3_TH_SMD, B.Cu at (60.6, 139.3)
- added D12: DIODE, kbd:D3_TH_SMD, B.Cu at (67.6, 157.4)
- added D13: DIODE, kbd:D3_TH_SMD, B.Cu at (92.0, 53.1)
- added D14: DIODE, kbd:D3_TH_SMD, B.Cu at (85.2, 73.2)
- added D15: DIODE, kbd:D3_TH_SMD, B.Cu at (85.5, 93.7)
- added D16: DIODE, kbd:D3_TH_SMD, B.Cu at (82.9, 113.1)
- added D17: DIODE, kbd:D3_TH_SMD, B.Cu at (79.9, 134.2)
- added D18: DIODE, kbd:D3_TH_SMD, B.Cu at (87.0, 152.0)
- added D19: DIODE, kbd:D3_TH_SMD, B.Cu at (110.8, 49.9)
- added D2: DIODE, kbd:D3_TH_SMD, B.Cu at (47.1, 82.3)
- added D20: DIODE, kbd:D3_TH_SMD, B.Cu at (105.2, 69.1)
- added D21: DIODE, kbd:D3_TH_SMD, B.Cu at (106.7, 88.6)
- added D22: DIODE, kbd:D3_TH_SMD, B.Cu at (102.8, 109.1)
- added D23: DIODE, kbd:D3_TH_SMD, B.Cu at (99.4, 129.4)
- added D24: DIODE, kbd:D3_TH_SMD, B.Cu at (107.0, 147.8)
- added D25: DIODE, kbd:D3_TH_SMD, B.Cu at (114.2, 49.8)
- added D26: DIODE, kbd:D3_TH_SMD, B.Cu at (126.1, 67.9)
- added D27: DIODE, kbd:D3_TH_SMD, B.Cu at (127.9, 88.6)
- added D28: DIODE, kbd:D3_TH_SMD, B.Cu at (124.1, 107.9)
- added D29: DIODE, kbd:D3_TH_SMD, B.Cu at (120.2, 127.0)
- added D3: DIODE, kbd:D3_TH_SMD, B.Cu at (48.3, 103.9)
- added D30: DIODE, kbd:D3_TH_SMD, B.Cu at (130.5, 149.6)
- added D31: DIODE, kbd:D3_TH_SMD, B.Cu at (135.1, 48.0)
- added D32: DIODE, kbd:D3_TH_SMD, B.Cu at (130.4, 67.5)
- added D33: DIODE, kbd:D3_TH_SMD, B.Cu at (130.9, 88.8)
- added D34: DIODE, kbd:D3_TH_SMD, B.Cu at (128.3, 107.8)
- added D35: DIODE, kbd:D3_TH_SMD, B.Cu at (124.2, 127.6)
- added D36: DIODE, kbd:D3_TH_SMD, B.Cu at (135.4, 151.6)
- added D37: DIODE, kbd:D3_TH_SMD, B.Cu at (155.6, 53.9)
- added D38: DIODE, kbd:D3_TH_SMD, B.Cu at (150.3, 72.5)
- added D39: DIODE, kbd:D3_TH_SMD, B.Cu at (153.2, 92.8)
- added D4: DIODE, kbd:D3_TH_SMD, B.Cu at (45.1, 123.7)
- added D40: DIODE, kbd:D3_TH_SMD, B.Cu at (148.0, 115.2)
- added D41: DIODE, kbd:D3_TH_SMD, B.Cu at (146.0, 134.9)
- added D42: DIODE, kbd:D3_TH_SMD, B.Cu at (155.0, 165.1)
- added D43: DIODE, kbd:D3_TH_SMD, B.Cu at (211.2, 83.4)
- added D44: DIODE, kbd:D3_TH_SMD, B.Cu at (193.8, 71.1)
- added D45: DIODE, kbd:D3_TH_SMD, B.Cu at (174.8, 63.0)
- added D46: DIODE, kbd:D3_TH_SMD, B.Cu at (169.6, 81.6)
- added D47: DIODE, kbd:D3_TH_SMD, B.Cu at (188.6, 90.5)
- added D48: DIODE, kbd:D3_TH_SMD, B.Cu at (170.3, 103.3)
- added D49: DIODE, kbd:D3_TH_SMD, B.Cu at (219.5, 82.7)
- added D5: DIODE, kbd:D3_TH_SMD, B.Cu at (42.2, 145.5)
- added D50: DIODE, kbd:D3_TH_SMD, B.Cu at (235.5, 99.4)
- added D51: DIODE, kbd:D3_TH_SMD, B.Cu at (227.0, 98.2)
- added D52: DIODE, kbd:D3_TH_SMD, B.Cu at (206.3, 104.9)
- added D53: DIODE, kbd:D3_TH_SMD, B.Cu at (189.1, 116.2)
- added D54: DIODE, kbd:D3_TH_SMD, B.Cu at (168.3, 124.4)
- added D55: DIODE, kbd:D3_TH_SMD, B.Cu at (247.7, 116.1)
- added D56: DIODE, kbd:D3_TH_SMD, B.Cu at (240.0, 114.2)
- added D57: DIODE, kbd:D3_TH_SMD, B.Cu at (219.8, 120.3)
- added D58: DIODE, kbd:D3_TH_SMD, B.Cu at (203.2, 131.5)
- added D59: DIODE, kbd:D3_TH_SMD, B.Cu at (185.4, 139.8)
- added D6: DIODE, kbd:D3_TH_SMD, B.Cu at (48.8, 163.2)
- added D60: DIODE, kbd:D3_TH_SMD, B.Cu at (165.2, 147.6)
- added D61: DIODE, kbd:D3_TH_SMD, B.Cu at (250.5, 131.8)
- added D62: DIODE, kbd:D3_TH_SMD, B.Cu at (231.6, 137.6)
- added D63: DIODE, kbd:D3_TH_SMD, B.Cu at (215.5, 148.8)
- added D64: DIODE, kbd:D3_TH_SMD, B.Cu at (197.8, 156.7)
- added D65: DIODE, kbd:D3_TH_SMD, B.Cu at (178.9, 164.6)
- added D66: DIODE, kbd:D3_TH_SMD, B.Cu at (151.4, 191.6)
- added D67: DIODE, kbd:D3_TH_SMD, B.Cu at (259.9, 150.7)
- added D68: DIODE, kbd:D3_TH_SMD, B.Cu at (241.2, 156.1)
- added D69: DIODE, kbd:D3_TH_SMD, B.Cu at (224.7, 167.3)
- added D7: DIODE, kbd:D3_TH_SMD, B.Cu at (72.2, 57.9)
- added D70: DIODE, kbd:D3_TH_SMD, B.Cu at (208.0, 175.7)
- added D71: DIODE, kbd:D3_TH_SMD, B.Cu at (189.6, 183.7)
- added D72: DIODE, kbd:D3_TH_SMD, B.Cu at (167.5, 206.3)
- added D73: DIODE, kbd:D3_TH_SMD, B.Cu at (267.1, 169.6)
- added D74: DIODE, kbd:D3_TH_SMD, B.Cu at (248.9, 175.3)
- added D75: DIODE, kbd:D3_TH_SMD, B.Cu at (232.1, 186.8)
- added D76: DIODE, kbd:D3_TH_SMD, B.Cu at (213.9, 195.3)
- added D77: DIODE, kbd:D3_TH_SMD, B.Cu at (196.4, 203.1)
- added D78: DIODE, kbd:D3_TH_SMD, B.Cu at (169.6, 208.9)
- added D79: DIODE, kbd:D3_TH_SMD, B.Cu at (272.4, 189.2)
- added D8: DIODE, kbd:D3_TH_SMD, B.Cu at (66.0, 77.1)
- added D80: DIODE, kbd:D3_TH_SMD, B.Cu at (254.3, 194.8)
- added D81: DIODE, kbd:D3_TH_SMD, B.Cu at (237.0, 206.7)
- added D82: DIODE, kbd:D3_TH_SMD, B.Cu at (219.0, 214.9)
- added D83: DIODE, kbd:D3_TH_SMD, B.Cu at (199.5, 223.6)
- added D84: DIODE, kbd:D3_TH_SMD, B.Cu at (180.0, 229.7)
- added D85: DIODE, kbd:D3_TH_SMD, B.Cu at (276.5, 208.8)
- added D86: DIODE, kbd:D3_TH_SMD, B.Cu at (257.7, 215.2)
- added D87: DIODE, kbd:D3_TH_SMD, B.Cu at (240.8, 226.5)
- added D88: DIODE, kbd:D3_TH_SMD, B.Cu at (222.9, 234.9)
- added D89: DIODE, kbd:D3_TH_SMD, B.Cu at (201.6, 243.9)
- added D9: DIODE, kbd:D3_TH_SMD, B.Cu at (66.9, 98.7)
- added D90: DIODE, kbd:D3_TH_SMD, B.Cu at (184.2, 251.3)
- added HOLE1: Val**, kbd:HOLE, F.Cu at (35.3, 45.5)
- added HOLE2: Val**, kbd:HOLE, F.Cu at (32.6, 186.8)
- added HOLE3: Val**, kbd:HOLE, F.Cu at (202.3, 64.5)
- added HOLE4: Val**, kbd:HOLE, F.Cu at (142.1, 176.7)
- added HOLE5: Val**, kbd:HOLE, F.Cu at (293.1, 220.4)
- added HOLE6: Val**, kbd:HOLE, F.Cu at (171.1, 274.4)
- added SW42: SW_PUSH, kbd:CherryMX_Hotswap_edit_wakunasi, F.Cu at (157.6, 176.3)
- added SW43: SW_PUSH, kbd:CherryMX_Hotswap_edit_wakunasi, F.Cu at (215.7, 94.1)
- added SW44: SW_PUSH, kbd:CherryMX_Hotswap_edit_wakunasi, F.Cu at (199.4, 80.9)
- added SW45: SW_PUSH, kbd:CherryMX_Hotswap_edit_wakunasi, F.Cu at (182.3, 70.5)
- added SW46: SW_PUSH, kbd:CherryMX_Hotswap_edit_wakunasi, F.Cu at (176.5, 90.2)
- added SW47: SW_PUSH, kbd:CherryMX_Hotswap_edit_wakunasi, F.Cu at (193.6, 101.2)
- added SW48: SW_PUSH, kbd:CherryMX_Hotswap_edit_wakunasi, F.Cu at (176.4, 113.2)
- added SW49: SW_PUSH, kbd:ResetSW_wakunasi, F.Cu at (227.4, 89.2)
- added SW50: SW_PUSH, kbd:ResetSW_wakunasi, F.Cu at (241.7, 106.4)
- added SW51: SW_PUSH, kbd:CherryMX_Hotswap_edit_wakunasi, F.Cu at (229.5, 109.6)
- added SW52: SW_PUSH, kbd:CherryMX_Hotswap_edit_wakunasi, F.Cu at (209.2, 116.0)
- added SW53: SW_PUSH, kbd:CherryMX_Hotswap_edit_wakunasi, F.Cu at (192.8, 126.9)
- added SW54: SW_PUSH, kbd:CherryMX_Hotswap_edit_wakunasi, F.Cu at (173.1, 135.4)
- added SW55: SW_PUSH, kbd:ResetSW_wakunasi, F.Cu at (253.1, 123.6)
- added SW56: SW_PUSH, kbd:CherryMX_Hotswap_edit_wakunasi, F.Cu at (240.9, 126.0)
- added SW57: SW_PUSH, kbd:CherryMX_Hotswap_edit_wakunasi, F.Cu at (221.3, 131.9)
- added SW58: SW_PUSH, kbd:CherryMX_Hotswap_edit_wakunasi, F.Cu at (205.3, 142.7)
- added SW59: SW_PUSH, kbd:CherryMX_Hotswap_edit_wakunasi, F.Cu at (187.6, 151.0)
- added SW60: SW_PUSH, kbd:CherryMX_Hotswap_edit_wakunasi, F.Cu at (168.7, 158.6)
- added SW61: SW_PUSH, kbd:CherryMX_Hotswap_edit_wakunasi, F.Cu at (250.7, 143.5)
- added SW62: SW_PUSH, kbd:CherryMX_Hotswap_edit_wakunasi, F.Cu at (231.9, 149.2)
- added SW63: SW_PUSH, kbd:CherryMX_Hotswap_edit_wakunasi, F.Cu at (215.8, 160.2)
- added SW64: SW_PUSH, kbd:CherryMX_Hotswap_edit_wakunasi, F.Cu at (198.4, 168.5)
- added SW65: SW_PUSH, kbd:CherryMX_Hotswap_edit_wakunasi, F.Cu at (180.4, 176.1)
- added SW66: SW_PUSH, kbd:CherryMX_Hotswap_edit_wakunasi, F.Cu at (139.8, 190.1)
- added SW67: SW_PUSH, kbd:CherryMX_Hotswap_edit_wakunasi, F.Cu at (258.9, 162.1)
- added SW68: SW_PUSH, kbd:CherryMX_Hotswap_edit_wakunasi, F.Cu at (240.3, 167.8)
- added SW69: SW_PUSH, kbd:CherryMX_Hotswap_edit_wakunasi, F.Cu at (223.8, 179.0)
- added SW70: SW_PUSH, kbd:CherryMX_Hotswap_edit_wakunasi, F.Cu at (206.3, 187.4)
- added SW71: SW_PUSH, kbd:CherryMX_Hotswap_edit_wakunasi, F.Cu at (188.5, 195.2)
- added SW72: SW_PUSH, kbd:CherryMX_Hotswap_edit_wakunasi, F.Cu at (156.8, 202.5)
- added SW73: SW_PUSH, kbd:CherryMX_Hotswap_edit_wakunasi, F.Cu at (265.1, 181.0)
- added SW74: SW_PUSH, kbd:CherryMX_Hotswap_edit_wakunasi, F.Cu at (246.6, 186.7)
- added SW75: SW_PUSH, kbd:CherryMX_Hotswap_edit_wakunasi, F.Cu at (229.6, 198.3)
- added SW76: SW_PUSH, kbd:CherryMX_Hotswap_edit_wakunasi, F.Cu at (211.8, 206.5)
- added SW77: SW_PUSH, kbd:CherryMX_Hotswap_edit_wakunasi, F.Cu at (193.7, 214.4)
- added SW78: SW_PUSH, kbd:CherryMX_Hotswap_edit_wakunasi, F.Cu at (170.4, 220.0)
- added SW79: SW_PUSH, kbd:CherryMX_Hotswap_edit_wakunasi, F.Cu at (269.9, 200.1)
- added SW80: SW_PUSH, kbd:CherryMX_Hotswap_edit_wakunasi, F.Cu at (251.3, 206.1)
- added SW81: SW_PUSH, kbd:CherryMX_Hotswap_edit_wakunasi, F.Cu at (233.9, 217.6)
- added SW82: SW_PUSH, kbd:CherryMX_Hotswap_edit_wakunasi, F.Cu at (215.6, 225.8)
- added SW83: SW_PUSH, kbd:CherryMX_Hotswap_edit_wakunasi, F.Cu at (197.1, 234.2)
- added SW84: SW_PUSH, kbd:CherryMX_Hotswap_edit_wakunasi, F.Cu at (177.6, 240.9)
- added SW85: SW_PUSH, kbd:CherryMX_Hotswap_edit_wakunasi, F.Cu at (273.4, 219.4)
- added SW86: SW_PUSH, kbd:CherryMX_Hotswap_edit_wakunasi, F.Cu at (255.0, 225.6)
- added SW87: SW_PUSH, kbd:CherryMX_Hotswap_edit_wakunasi, F.Cu at (237.0, 237.2)
- added SW88: SW_PUSH, kbd:CherryMX_Hotswap_edit_wakunasi, F.Cu at (218.1, 245.6)
- added SW89: SW_PUSH, kbd:CherryMX_Hotswap_edit_wakunasi, F.Cu at (198.9, 254.1)
- added SW90: SW_PUSH, kbd:CherryMX_Hotswap_edit_wakunasi, F.Cu at (179.3, 261.8)
- added SW91: SW_PUSH, kbd:ResetSW_wakunasi, F.Cu at (60.0, 49.1)
- added SW92: SW_PUSH, kbd:ResetSW_wakunasi, F.Cu at (80.7, 44.5)
- added SW93: SW_SPDT, kbd:SW_Slide_edit_wakunasi, F.Cu at (210.9, 70.6)
- added U2: ProMicro, kbd:ProMicro_v3.6, B.Cu at (111.0, 28.1)
- added U3: 74HC595, kbd:SN74HC595_DIP-16_W7.62mm_Socket_2, F.Cu at (142.5, 35.7)
- added U4: 74HC595, kbd:SN74HC595_DIP-16_W7.62mm_Socket_2, F.Cu at (163.1, 40.1)
- added U5: 74HC595, kbd:SN74HC595_DIP-16_W7.62mm_Socket_2, B.Cu at (144.6, 33.1)
- added U6: 74HC595, kbd:SN74HC595_DIP-16_W7.62mm_Socket_2, B.Cu at (165.3, 37.5)
- J2: value Conn_01x01_Female -> Pi; footprint Connector_Pin:Pin_D1.0mm_L10.0mm -> kbd:PinSocket_2x20_P2.54mm_Vertical_edit_wakunasi
- SW1, SW11, SW12, SW13, SW14, SW16, SW17, SW18, SW19, SW2, SW20, SW21, SW22, SW23, SW24, SW25, SW26, SW27, SW28, SW29, SW3, SW30, SW31, SW32, SW33, SW34, SW35, SW36, SW37, SW38, SW39, SW4, SW40, SW6, SW7, SW8, SW9: value SW_PUSH-kbd -> SW_PUSH; footprint kbd:CherryMX_MidHeight_Hotswap_edit -> kbd:CherryMX_Hotswap_edit_wakunasi
- SW10, SW15, SW5: value SW_PUSH-kbd -> SW_PUSH; footprint kbd:ResetSW_with_diode -> kbd:CherryMX_Hotswap_edit_wakunasi
- SW41: footprint kbd:ResetSW -> kbd:CherryMX_Hotswap_edit_wakunasi
- U1: value BluePill_STM32F103C -> ProMicro; footprint BluePill_breakouts:BluePill_STM32F103C_0.9_Double -> kbd:ProMicro_v3.6
- moved SW36 143.7 mm to (141.6, 160.8), turned to 326 degrees
- moved SW6 139.7 mm to (41.4, 171.5), turned to 20 degrees
- moved SW11 123.4 mm to (52.8, 147.0)
- moved SW12 119.3 mm to (59.8, 165.1), turned to 18 degrees
- moved SW41 102.9 mm to (152.5, 144.4), turned to 326 degrees
- moved SW17 101.7 mm to (71.4, 141.3), turned to 16 degrees
- moved SW16 101.6 mm to (74.5, 120.5), turned to 15 degrees
- moved SW18 100.5 mm to (78.5, 159.4), turned to 16 degrees
- moved SW5 99.6 mm to (34.3, 153.5), turned to 21 degrees
- moved SW23 81.4 mm to (90.5, 136.4), turned to 13 degrees
- moved SW22 80.1 mm to (93.7, 116.0), turned to 12 degrees
- moved SW21 79.5 mm to (96.6, 95.7), turned to 11 degrees
- moved SW24 78.9 mm to (97.7, 154.6), turned to 12 degrees
- moved U1 73.4 mm to (109.8, 30.6), turned to 90 degrees
- moved SW30 72.1 mm to (119.5, 153.2), turned to 355 degrees
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Connections:
- J2 pad 1: Net-(J2-Pad1) -> (no net)
- SW1 pad 1: col00 -> (no net)
- SW1 pad 2: Net-(SW1-Pad2) -> (no net)
- SW10 pad 1: col01 -> (no net)
- SW10 pad 2: Net-(SW10-Pad2) -> (no net)
- SW11 pad 1: col02 -> (no net)
- SW11 pad 2: Net-(SW11-Pad2) -> (no net)
- SW12 pad 1: col02 -> (no net)
- SW12 pad 2: Net-(SW12-Pad2) -> (no net)
- SW13 pad 1: col02 -> (no net)
- SW13 pad 2: Net-(SW13-Pad2) -> (no net)
- SW14 pad 1: col02 -> (no net)
- SW14 pad 2: Net-(SW14-Pad2) -> (no net)
- SW15 pad 1: col02 -> (no net)
- SW15 pad 2: Net-(SW15-Pad2) -> (no net)
- SW16 pad 1: col03 -> (no net)
- SW16 pad 2: Net-(SW16-Pad2) -> (no net)
- SW17 pad 1: col03 -> (no net)
- SW17 pad 2: Net-(SW17-Pad2) -> (no net)
- SW18 pad 1: col03 -> (no net)
- SW18 pad 2: Net-(SW18-Pad2) -> (no net)
- SW19 pad 1: col03 -> (no net)
- SW19 pad 2: Net-(SW19-Pad2) -> (no net)
- SW2 pad 1: col00 -> (no net)
- SW2 pad 2: Net-(SW2-Pad2) -> (no net)
- SW20 pad 1: col03 -> (no net)
- SW20 pad 2: Net-(SW20-Pad2) -> (no net)
- SW21 pad 1: col04 -> (no net)
- SW21 pad 2: Net-(SW21-Pad2) -> (no net)
- SW22 pad 1: col04 -> (no net)
- SW22 pad 2: Net-(SW22-Pad2) -> (no net)
- SW23 pad 1: col04 -> (no net)
- SW23 pad 2: Net-(SW23-Pad2) -> (no net)
- SW24 pad 1: col04 -> (no net)
- SW24 pad 2: Net-(SW24-Pad2) -> (no net)
- SW25 pad 1: col04 -> (no net)
- SW25 pad 2: Net-(SW25-Pad2) -> (no net)
- SW26 pad 1: col05 -> (no net)
- SW26 pad 2: Net-(SW26-Pad2) -> (no net)
- SW27 pad 1: col05 -> (no net)
- SW27 pad 2: Net-(SW27-Pad2) -> (no net)
- SW28 pad 1: col05 -> (no net)
- SW28 pad 2: Net-(SW28-Pad2) -> (no net)
- SW29 pad 1: col05 -> (no net)
- SW29 pad 2: Net-(SW29-Pad2) -> (no net)
- SW3 pad 1: col00 -> (no net)
- SW3 pad 2: Net-(SW3-Pad2) -> (no net)
- SW30 pad 1: col05 -> (no net)
- SW30 pad 2: Net-(SW30-Pad2) -> (no net)
- SW31 pad 1: col06 -> (no net)
- SW31 pad 2: Net-(SW31-Pad2) -> (no net)
- SW32 pad 1: col06 -> (no net)
- SW32 pad 2: Net-(SW32-Pad2) -> (no net)
- SW33 pad 1: col06 -> (no net)
- SW33 pad 2: Net-(SW33-Pad2) -> (no net)
- SW34 pad 1: col06 -> (no net)
- SW34 pad 2: Net-(SW34-Pad2) -> (no net)
- SW35 pad 1: col06 -> (no net)
- SW35 pad 2: Net-(SW35-Pad2) -> (no net)
- SW36 pad 1: col07 -> (no net)
- SW36 pad 2: Net-(SW36-Pad2) -> (no net)
- SW37 pad 1: col07 -> (no net)
- SW37 pad 2: Net-(SW37-Pad2) -> (no net)
- SW38 pad 1: col07 -> (no net)
- SW38 pad 2: Net-(SW38-Pad2) -> (no net)
- SW39 pad 1: col07 -> (no net)
- SW39 pad 2: Net-(SW39-Pad2) -> (no net)
- SW4 pad 1: col00 -> (no net)
- SW4 pad 2: Net-(SW4-Pad2) -> (no net)
- SW40 pad 1: col07 -> (no net)
- SW40 pad 2: Net-(SW40-Pad2) -> (no net)
- SW41 pad 1: hardware_reset -> (no net)
- SW41 pad 2: GND -> (no net)
- SW5 pad 1: col00 -> (no net)
- SW5 pad 2: Net-(SW5-Pad2) -> (no net)
- SW6 pad 1: col01 -> (no net)
- SW6 pad 2: Net-(SW6-Pad2) -> (no net)
- SW7 pad 1: col01 -> (no net)
- SW7 pad 2: Net-(SW7-Pad2) -> (no net)
- SW8 pad 1: col01 -> (no net)
- SW8 pad 2: Net-(SW8-Pad2) -> (no net)
- SW9 pad 1: col01 -> (no net)
- SW9 pad 2: Net-(SW9-Pad2) -> (no net)
- U1 pad 1: Net-(U1-Pad1) -> (no net)
- U1 pad 10: col02 -> (no net)
- U1 pad 11: col03 -> (no net)
- U1 pad 12: col00 -> (no net)
- U1 pad 13: col04 -> (no net)
- U1 pad 14: col05 -> (no net)
- U1 pad 15: Net-(U1-Pad15) -> (no net)
- U1 pad 16: Net-(U1-Pad16) -> (no net)
- U1 pad 17: hardware_reset -> (no net)
- U1 pad 18: VCC -> (no net)
- U1 pad 19: GND -> (no net)
- U1 pad 2: Net-(U1-Pad2) -> (no net)
- U1 pad 20: GND -> (no net)
- U1 pad 21: Net-(U1-Pad21) -> (no net)
- U1 pad 22: Net-(U1-Pad22) -> (no net)
- U1 pad 23: Net-(U1-Pad23) -> (no net)
- U1 pad 24: Net-(U1-Pad24) -> (no net)
- U1 pad 3: Net-(U1-Pad3) -> (no net)
- U1 pad 4: Net-(U1-Pad4) -> (no net)
- U1 pad 5: col07 -> (no net)
- U1 pad 6: col06 -> (no net)
- U1 pad 7: Net-(J2-Pad1) -> (no net)
- U1 pad 8: Net-(J3-Pad1) -> (no net)
- U1 pad 9: col01 -> (no net)
Routing:
- net (no net): track 0.00 -> 11725.6 mm, vias 2 -> 448
- net row04: track 421.4 -> 0.00 mm, vias 1 -> 0
- net col03: track 352.2 -> 0.00 mm, vias 1 -> 0
- net col00: track 344.0 -> 0.00 mm
- net col01: track 331.5 -> 0.00 mm, vias 1 -> 0
- net col02: track 331.3 -> 0.00 mm, vias 1 -> 0
- net col04: track 323.5 -> 0.00 mm, vias 1 -> 0
- net col07: track 312.8 -> 0.00 mm, vias 1 -> 0
- net col06: track 291.8 -> 0.00 mm, vias 1 -> 0
- net col05: track 287.5 -> 0.00 mm, vias 1 -> 0
- net row00: track 235.9 -> 0.00 mm, vias 1 -> 0
- net row03: track 232.9 -> 0.00 mm, vias 1 -> 0
- net row02: track 221.7 -> 0.00 mm
- net row01: track 212.3 -> 0.00 mm
- net VCC: track 101.3 -> 0.00 mm, vias 3 -> 0
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- added copper zone on B.Cu, net (none)
- added copper zone on F.Cu, net (none)
- removed copper zone on B.Cu, net GND
- removed copper zone on F.Cu, net GND
Other:
- board size 212.8 x 143.6 mm -> 290.9 x 267.8 mm
- board text removed: "Fan74 v1.0 Designed by H&C 20200314"

Commit message: うごかない
Parts:
- J2: footprint kbd:PinSocket_2x20_P2.54mm_Vertical_edit_wakunasi -> Connector_PinSocket_2.54mm:PinSocket_2x20_P2.54mm_Vertical
- SW1, SW10, SW11, SW12, SW13, SW14, SW15, SW16, SW17, SW18, SW19, SW2, SW20, SW21, SW22, SW23, SW24, SW25, SW26, SW27, SW28, SW29, SW3, SW30, SW31, SW32, SW33, SW34, SW35, SW36, SW37, SW38, SW39, SW4, SW40, SW41, SW42, SW43, SW44, SW45, SW46, SW47, SW48, SW5, SW51, SW52, SW53, SW54, SW56, SW57, SW58, SW59, SW6, SW60, SW61, SW62, SW63, SW64, SW65, SW66, SW67, SW68, SW69, SW7, SW70, SW71, SW72, SW73, SW74, SW75, SW76, SW77, SW78, SW79, SW8, SW80, SW81, SW82, SW83, SW84, SW85, SW86, SW87, SW88, SW89, SW9, SW90: footprint kbd:CherryMX_Hotswap_edit_wakunasi -> kbd:CherryMX_Hotswap
- SW49, SW50, SW55, SW91, SW92: footprint kbd:ResetSW_wakunasi -> kbd:ResetSW
- SW93: footprint kbd:SW_Slide_edit_wakunasi -> Button_Switch_THT:SW_Slide_1P2T_CK_OS102011MS2Q
Connections:
- D1 pad 1: (no net) -> row00
- D1 pad 2: (no net) -> Net-(D1-Pad2)
- D10 pad 1: (no net) -> row03
- D10 pad 2: (no net) -> Net-(D10-Pad2)
- D11 pad 1: (no net) -> row04
- D11 pad 2: (no net) -> Net-(D11-Pad2)
- D12 pad 1: (no net) -> row05
- D12 pad 2: (no net) -> Net-(D12-Pad2)
- D13 pad 1: (no net) -> row00
- D13 pad 2: (no net) -> Net-(D13-Pad2)
- D14 pad 1: (no net) -> row01
- D14 pad 2: (no net) -> Net-(D14-Pad2)
- D15 pad 1: (no net) -> row02
- D15 pad 2: (no net) -> Net-(D15-Pad2)
- D16 pad 1: (no net) -> row03
- D16 pad 2: (no net) -> Net-(D16-Pad2)
- D17 pad 1: (no net) -> row04
- D17 pad 2: (no net) -> Net-(D17-Pad2)
- D18 pad 1: (no net) -> row05
- D18 pad 2: (no net) -> Net-(D18-Pad2)
- D19 pad 1: (no net) -> row00
- D19 pad 2: (no net) -> Net-(D19-Pad2)
- D2 pad 1: (no net) -> row01
- D2 pad 2: (no net) -> Net-(D2-Pad2)
- D20 pad 1: (no net) -> row01
- D20 pad 2: (no net) -> Net-(D20-Pad2)
- D21 pad 1: (no net) -> row02
- D21 pad 2: (no net) -> Net-(D21-Pad2)
- D22 pad 1: (no net) -> row03
- D22 pad 2: (no net) -> Net-(D22-Pad2)
- D23 pad 1: (no net) -> row04
- D23 pad 2: (no net) -> Net-(D23-Pad2)
- D24 pad 1: (no net) -> row05
- D24 pad 2: (no net) -> Net-(D24-Pad2)
- D25 pad 1: (no net) -> row00
- D25 pad 2: (no net) -> Net-(D25-Pad2)
- D26 pad 1: (no net) -> row01
- D26 pad 2: (no net) -> Net-(D26-Pad2)
- D27 pad 1: (no net) -> row02
- D27 pad 2: (no net) -> Net-(D27-Pad2)
- D28 pad 1: (no net) -> row03
- D28 pad 2: (no net) -> Net-(D28-Pad2)
- D29 pad 1: (no net) -> row04
- D29 pad 2: (no net) -> Net-(D29-Pad2)
- D3 pad 1: (no net) -> row02
- D3 pad 2: (no net) -> Net-(D3-Pad2)
- D30 pad 1: (no net) -> row05
- D30 pad 2: (no net) -> Net-(D30-Pad2)
- D31 pad 1: (no net) -> row00
- D31 pad 2: (no net) -> Net-(D31-Pad2)
- D32 pad 1: (no net) -> row01
- D32 pad 2: (no net) -> Net-(D32-Pad2)
- D33 pad 1: (no net) -> row02
- D33 pad 2: (no net) -> Net-(D33-Pad2)
- D34 pad 1: (no net) -> row03
- D34 pad 2: (no net) -> Net-(D34-Pad2)
- D35 pad 1: (no net) -> row04
- D35 pad 2: (no net) -> Net-(D35-Pad2)
- D36 pad 1: (no net) -> row05
- D36 pad 2: (no net) -> Net-(D36-Pad2)
- D37 pad 1: (no net) -> row00
- D37 pad 2: (no net) -> Net-(D37-Pad2)
- D38 pad 1: (no net) -> row01
- D38 pad 2: (no net) -> Net-(D38-Pad2)
- D39 pad 1: (no net) -> row02
- D39 pad 2: (no net) -> Net-(D39-Pad2)
- D4 pad 1: (no net) -> row03
- D4 pad 2: (no net) -> Net-(D4-Pad2)
- D40 pad 1: (no net) -> row03
- D40 pad 2: (no net) -> Net-(D40-Pad2)
- D41 pad 1: (no net) -> row04
- D41 pad 2: (no net) -> Net-(D41-Pad2)
- D42 pad 1: (no net) -> row05
- D42 pad 2: (no net) -> Net-(D42-Pad2)
- D43 pad 1: (no net) -> row00
- D43 pad 2: (no net) -> Net-(D43-Pad2)
- D44 pad 1: (no net) -> row01
- D44 pad 2: (no net) -> Net-(D44-Pad2)
- D45 pad 1: (no net) -> row02
- D45 pad 2: (no net) -> Net-(D45-Pad2)
- D46 pad 1: (no net) -> row03
- D46 pad 2: (no net) -> Net-(D46-Pad2)
- D47 pad 1: (no net) -> row04
- D47 pad 2: (no net) -> Net-(D47-Pad2)
- D48 pad 1: (no net) -> row05
- D48 pad 2: (no net) -> Net-(D48-Pad2)
- D49 pad 1: (no net) -> row00
- D49 pad 2: (no net) -> Net-(D49-Pad2)
- D5 pad 1: (no net) -> row04
- D5 pad 2: (no net) -> Net-(D5-Pad2)
- D50 pad 1: (no net) -> row01
- D50 pad 2: (no net) -> Net-(D50-Pad2)
- D51 pad 1: (no net) -> row02
- D51 pad 2: (no net) -> Net-(D51-Pad2)
- D52 pad 1: (no net) -> row03
- D52 pad 2: (no net) -> Net-(D52-Pad2)
- D53 pad 1: (no net) -> row04
- D53 pad 2: (no net) -> Net-(D53-Pad2)
- D54 pad 1: (no net) -> row05
- D54 pad 2: (no net) -> Net-(D54-Pad2)
- D55 pad 1: (no net) -> row00
- D55 pad 2: (no net) -> Net-(D55-Pad2)
- D56 pad 1: (no net) -> row01
- D56 pad 2: (no net) -> Net-(D56-Pad2)
- D57 pad 1: (no net) -> row02
- D57 pad 2: (no net) -> Net-(D57-Pad2)
- D58 pad 1: (no net) -> row03
- D58 pad 2: (no net) -> Net-(D58-Pad2)
- D59 pad 1: (no net) -> row04
- D59 pad 2: (no net) -> Net-(D59-Pad2)
- D6 pad 1: (no net) -> row05
- D6 pad 2: (no net) -> Net-(D6-Pad2)
- D60 pad 1: (no net) -> row05
- D60 pad 2: (no net) -> Net-(D60-Pad2)
- D61 pad 1: (no net) -> row00
- D61 pad 2: (no net) -> Net-(D61-Pad2)
- D62 pad 1: (no net) -> row01
- D62 pad 2: (no net) -> Net-(D62-Pad2)
- D63 pad 1: (no net) -> row02
- D63 pad 2: (no net) -> Net-(D63-Pad2)
- D64 pad 1: (no net) -> row03
- D64 pad 2: (no net) -> Net-(D64-Pad2)
- D65 pad 1: (no net) -> row04
- D65 pad 2: (no net) -> Net-(D65-Pad2)
- D66 pad 1: (no net) -> row05
- D66 pad 2: (no net) -> Net-(D66-Pad2)
- D67 pad 1: (no net) -> row00
- D67 pad 2: (no net) -> Net-(D67-Pad2)
- D68 pad 1: (no net) -> row01
- D68 pad 2: (no net) -> Net-(D68-Pad2)
- D69 pad 1: (no net) -> row02
- D69 pad 2: (no net) -> Net-(D69-Pad2)
- D7 pad 1: (no net) -> row00
- D7 pad 2: (no net) -> Net-(D7-Pad2)
- D70 pad 1: (no net) -> row03
- D70 pad 2: (no net) -> Net-(D70-Pad2)
- D71 pad 1: (no net) -> row04
- D71 pad 2: (no net) -> Net-(D71-Pad2)
- D72 pad 1: (no net) -> row05
- D72 pad 2: (no net) -> Net-(D72-Pad2)
- D73 pad 1: (no net) -> row00
- D73 pad 2: (no net) -> Net-(D73-Pad2)
- D74 pad 1: (no net) -> row01
- D74 pad 2: (no net) -> Net-(D74-Pad2)
- D75 pad 1: (no net) -> row02
- D75 pad 2: (no net) -> Net-(D75-Pad2)
- D76 pad 1: (no net) -> row03
- D76 pad 2: (no net) -> Net-(D76-Pad2)
- D77 pad 1: (no net) -> row04
- D77 pad 2: (no net) -> Net-(D77-Pad2)
- D78 pad 1: (no net) -> row05
- D78 pad 2: (no net) -> Net-(D78-Pad2)
- D79 pad 1: (no net) -> row00
- D79 pad 2: (no net) -> Net-(D79-Pad2)
- D8 pad 1: (no net) -> row01
- D8 pad 2: (no net) -> Net-(D8-Pad2)
- D80 pad 1: (no net) -> row01
- D80 pad 2: (no net) -> Net-(D80-Pad2)
- D81 pad 1: (no net) -> row02
- D81 pad 2: (no net) -> Net-(D81-Pad2)
- D82 pad 1: (no net) -> row03
- D82 pad 2: (no net) -> Net-(D82-Pad2)
- D83 pad 1: (no net) -> row04
- D83 pad 2: (no net) -> Net-(D83-Pad2)
- D84 pad 1: (no net) -> row05
- D84 pad 2: (no net) -> Net-(D84-Pad2)
- D85 pad 1: (no net) -> row00
- D85 pad 2: (no net) -> Net-(D85-Pad2)
- D86 pad 1: (no net) -> row01
- D86 pad 2: (no net) -> Net-(D86-Pad2)
- D87 pad 1: (no net) -> row02
- D87 pad 2: (no net) -> Net-(D87-Pad2)
- D88 pad 1: (no net) -> row03
- D88 pad 2: (no net) -> Net-(D88-Pad2)
- D89 pad 1: (no net) -> row04
- D89 pad 2: (no net) -> Net-(D89-Pad2)
- D9 pad 1: (no net) -> row02
- D9 pad 2: (no net) -> Net-(D9-Pad2)
- D90 pad 1: (no net) -> row05
- D90 pad 2: (no net) -> Net-(D90-Pad2)
- J2 pad 1: (no net) -> Net-(J2-Pad1)
- J2 pad 10: (no net) -> Net-(J2-Pad10)
- J2 pad 11: (no net) -> Net-(J2-Pad11)
- J2 pad 12: (no net) -> Net-(J2-Pad12)
- J2 pad 13: (no net) -> Net-(J2-Pad13)
- J2 pad 14: (no net) -> Net-(J2-Pad14)
- J2 pad 15: (no net) -> Net-(J2-Pad15)
- J2 pad 16: (no net) -> Net-(J2-Pad16)
- J2 pad 17: (no net) -> Net-(J2-Pad17)
- J2 pad 18: (no net) -> Net-(J2-Pad18)
- J2 pad 19: (no net) -> Net-(J2-Pad19)
- J2 pad 2: (no net) -> Net-(J2-Pad2)
- J2 pad 20: (no net) -> Net-(J2-Pad20)
- J2 pad 21: (no net) -> Net-(J2-Pad21)
- J2 pad 22: (no net) -> Net-(J2-Pad22)
- J2 pad 23: (no net) -> Net-(J2-Pad23)
- J2 pad 24: (no net) -> Net-(J2-Pad24)
- J2 pad 25: (no net) -> Net-(J2-Pad25)
- J2 pad 26: (no net) -> Net-(J2-Pad26)
- J2 pad 27: (no net) -> Net-(J2-Pad27)
- J2 pad 28: (no net) -> Net-(J2-Pad28)
- J2 pad 29: (no net) -> Net-(J2-Pad29)
- J2 pad 3: (no net) -> Net-(J2-Pad3)
- J2 pad 30: (no net) -> Net-(J2-Pad30)
- J2 pad 31: (no net) -> Net-(J2-Pad31)
- J2 pad 32: (no net) -> Net-(J2-Pad32)
- J2 pad 33: (no net) -> Net-(J2-Pad33)
- J2 pad 34: (no net) -> Net-(J2-Pad34)
- J2 pad 35: (no net) -> Net-(J2-Pad35)
- J2 pad 36: (no net) -> GND
- J2 pad 37: (no net) -> Net-(J2-Pad37)
- J2 pad 38: (no net) -> Net-(J2-Pad38)
- J2 pad 39: (no net) -> Net-(J2-Pad39)
- J2 pad 4: (no net) -> Net-(J2-Pad4)
- J2 pad 40: (no net) -> Net-(J2-Pad38)
- J2 pad 5: (no net) -> Net-(J2-Pad5)
- J2 pad 6: (no net) -> Net-(J2-Pad6)
- J2 pad 7: (no net) -> Net-(J2-Pad7)
- J2 pad 8: (no net) -> Net-(J2-Pad8)
- J2 pad 9: (no net) -> Net-(J2-Pad9)
- SW1 pad 1: (no net) -> col00
- SW1 pad 2: (no net) -> Net-(D1-Pad2)
- SW10 pad 1: (no net) -> col01
- SW10 pad 2: (no net) -> Net-(D10-Pad2)
- SW11 pad 1: (no net) -> col01
- SW11 pad 2: (no net) -> Net-(D11-Pad2)
- SW12 pad 1: (no net) -> col01
- SW12 pad 2: (no net) -> Net-(D12-Pad2)
- SW13 pad 1: (no net) -> col02
- SW13 pad 2: (no net) -> Net-(D13-Pad2)
- SW14 pad 1: (no net) -> col02
- SW14 pad 2: (no net) -> Net-(D14-Pad2)
- SW15 pad 1: (no net) -> col02
- SW15 pad 2: (no net) -> Net-(D15-Pad2)
- SW16 pad 1: (no net) -> col02
- SW16 pad 2: (no net) -> Net-(D16-Pad2)
- SW17 pad 1: (no net) -> col02
- SW17 pad 2: (no net) -> Net-(D17-Pad2)
- SW18 pad 1: (no net) -> col02
- SW18 pad 2: (no net) -> Net-(D18-Pad2)
- SW19 pad 1: (no net) -> col03
- SW19 pad 2: (no net) -> Net-(D19-Pad2)
- SW2 pad 1: (no net) -> col00
- SW2 pad 2: (no net) -> Net-(D2-Pad2)
- SW20 pad 1: (no net) -> col03
- SW20 pad 2: (no net) -> Net-(D20-Pad2)
- SW21 pad 1: (no net) -> col03
- SW21 pad 2: (no net) -> Net-(D21-Pad2)
- SW22 pad 1: (no net) -> col03
- SW22 pad 2: (no net) -> Net-(D22-Pad2)
- SW23 pad 1: (no net) -> col03
- SW23 pad 2: (no net) -> Net-(D23-Pad2)
- SW24 pad 1: (no net) -> col03
- SW24 pad 2: (no net) -> Net-(D24-Pad2)
- SW25 pad 1: (no net) -> col04
- SW25 pad 2: (no net) -> Net-(D25-Pad2)
- SW26 pad 1: (no net) -> col04
- SW26 pad 2: (no net) -> Net-(D26-Pad2)
- SW27 pad 1: (no net) -> col04
- SW27 pad 2: (no net) -> Net-(D27-Pad2)
- SW28 pad 1: (no net) -> col04
- SW28 pad 2: (no net) -> Net-(D28-Pad2)
- SW29 pad 1: (no net) -> col04
- SW29 pad 2: (no net) -> Net-(D29-Pad2)
- SW3 pad 1: (no net) -> col00
- SW3 pad 2: (no net) -> Net-(D3-Pad2)
- SW30 pad 1: (no net) -> col04
- SW30 pad 2: (no net) -> Net-(D30-Pad2)
- SW31 pad 1: (no net) -> col05
- SW31 pad 2: (no net) -> Net-(D31-Pad2)
- SW32 pad 1: (no net) -> col05
- SW32 pad 2: (no net) -> Net-(D32-Pad2)
- SW33 pad 1: (no net) -> col05
- SW33 pad 2: (no net) -> Net-(D33-Pad2)
- SW34 pad 1: (no net) -> col05
- SW34 pad 2: (no net) -> Net-(D34-Pad2)
- SW35 pad 1: (no net) -> col05
- SW35 pad 2: (no net) -> Net-(D35-Pad2)
- SW36 pad 1: (no net) -> col05
- SW36 pad 2: (no net) -> Net-(D36-Pad2)
- SW37 pad 1: (no net) -> col06
- SW37 pad 2: (no net) -> Net-(D37-Pad2)
- SW38 pad 1: (no net) -> col06
- SW38 pad 2: (no net) -> Net-(D38-Pad2)
- SW39 pad 1: (no net) -> col06
- SW39 pad 2: (no net) -> Net-(D39-Pad2)
- SW4 pad 1: (no net) -> col00
- SW4 pad 2: (no net) -> Net-(D4-Pad2)
- SW40 pad 1: (no net) -> col06
- SW40 pad 2: (no net) -> Net-(D40-Pad2)
- SW41 pad 1: (no net) -> col06
- SW41 pad 2: (no net) -> Net-(D41-Pad2)
- SW42 pad 1: (no net) -> col06
- SW42 pad 2: (no net) -> Net-(D42-Pad2)
- SW43 pad 1: (no net) -> col07
- SW43 pad 2: (no net) -> Net-(D43-Pad2)
- SW44 pad 1: (no net) -> col07
- SW44 pad 2: (no net) -> Net-(D44-Pad2)
- SW45 pad 1: (no net) -> col07
- SW45 pad 2: (no net) -> Net-(D45-Pad2)
- SW46 pad 1: (no net) -> col07
- SW46 pad 2: (no net) -> Net-(D46-Pad2)
- SW47 pad 1: (no net) -> col07
- SW47 pad 2: (no net) -> Net-(D47-Pad2)
- SW48 pad 1: (no net) -> col07
- SW48 pad 2: (no net) -> Net-(D48-Pad2)
- SW49 pad 1: (no net) -> col08
- SW49 pad 2: (no net) -> Net-(D49-Pad2)
- SW5 pad 1: (no net) -> col00
- SW5 pad 2: (no net) -> Net-(D5-Pad2)
- SW50 pad 1: (no net) -> col08
- SW50 pad 2: (no net) -> Net-(D50-Pad2)
- SW51 pad 1: (no net) -> col08
- SW51 pad 2: (no net) -> Net-(D51-Pad2)
- SW52 pad 1: (no net) -> col08
- SW52 pad 2: (no net) -> Net-(D52-Pad2)
- SW53 pad 1: (no net) -> col08
- SW53 pad 2: (no net) -> Net-(D53-Pad2)
- SW54 pad 1: (no net) -> col08
- SW54 pad 2: (no net) -> Net-(D54-Pad2)
- SW55 pad 1: (no net) -> col09
- SW55 pad 2: (no net) -> Net-(D55-Pad2)
- SW56 pad 1: (no net) -> col09
- SW56 pad 2: (no net) -> Net-(D56-Pad2)
- SW57 pad 1: (no net) -> col09
- SW57 pad 2: (no net) -> Net-(D57-Pad2)
- SW58 pad 1: (no net) -> col09
- SW58 pad 2: (no net) -> Net-(D58-Pad2)
- SW59 pad 1: (no net) -> col09
- SW59 pad 2: (no net) -> Net-(D59-Pad2)
- SW6 pad 1: (no net) -> col00
- SW6 pad 2: (no net) -> Net-(D6-Pad2)
- SW60 pad 1: (no net) -> col09
- SW60 pad 2: (no net) -> Net-(D60-Pad2)
- SW61 pad 1: (no net) -> col10
- SW61 pad 2: (no net) -> Net-(D61-Pad2)
- SW62 pad 1: (no net) -> col10
- SW62 pad 2: (no net) -> Net-(D62-Pad2)
- SW63 pad 1: (no net) -> col10
- SW63 pad 2: (no net) -> Net-(D63-Pad2)
- SW64 pad 1: (no net) -> col10
- SW64 pad 2: (no net) -> Net-(D64-Pad2)
- SW65 pad 1: (no net) -> col10
- SW65 pad 2: (no net) -> Net-(D65-Pad2)
- SW66 pad 1: (no net) -> col10
- SW66 pad 2: (no net) -> Net-(D66-Pad2)
- SW67 pad 1: (no net) -> col11
- SW67 pad 2: (no net) -> Net-(D67-Pad2)
- SW68 pad 1: (no net) -> col11
- SW68 pad 2: (no net) -> Net-(D68-Pad2)
- SW69 pad 1: (no net) -> col11
- SW69 pad 2: (no net) -> Net-(D69-Pad2)
- SW7 pad 1: (no net) -> col01
- SW7 pad 2: (no net) -> Net-(D7-Pad2)
- SW70 pad 1: (no net) -> col11
- SW70 pad 2: (no net) -> Net-(D70-Pad2)
- SW71 pad 1: (no net) -> col11
- SW71 pad 2: (no net) -> Net-(D71-Pad2)
- SW72 pad 1: (no net) -> col11
- SW72 pad 2: (no net) -> Net-(D72-Pad2)
- SW73 pad 1: (no net) -> col12
- SW73 pad 2: (no net) -> Net-(D73-Pad2)
- SW74 pad 1: (no net) -> col12
- SW74 pad 2: (no net) -> Net-(D74-Pad2)
- SW75 pad 1: (no net) -> col12
- SW75 pad 2: (no net) -> Net-(D75-Pad2)
- SW76 pad 1: (no net) -> col12
- SW76 pad 2: (no net) -> Net-(D76-Pad2)
- SW77 pad 1: (no net) -> col12
- SW77 pad 2: (no net) -> Net-(D77-Pad2)
- SW78 pad 1: (no net) -> col12
- SW78 pad 2: (no net) -> Net-(D78-Pad2)
- SW79 pad 1: (no net) -> col13
- SW79 pad 2: (no net) -> Net-(D79-Pad2)
- SW8 pad 1: (no net) -> col01
- SW8 pad 2: (no net) -> Net-(D8-Pad2)
- SW80 pad 1: (no net) -> col13
- SW80 pad 2: (no net) -> Net-(D80-Pad2)
- SW81 pad 1: (no net) -> col13
- SW81 pad 2: (no net) -> Net-(D81-Pad2)
- SW82 pad 1: (no net) -> col13
- SW82 pad 2: (no net) -> Net-(D82-Pad2)
- SW83 pad 1: (no net) -> col13
- SW83 pad 2: (no net) -> Net-(D83-Pad2)
- SW84 pad 1: (no net) -> col13
- SW84 pad 2: (no net) -> Net-(D84-Pad2)
- SW85 pad 1: (no net) -> col14
- SW85 pad 2: (no net) -> Net-(D85-Pad2)
- SW86 pad 1: (no net) -> col14
- SW86 pad 2: (no net) -> Net-(D86-Pad2)
- SW87 pad 1: (no net) -> col14
- SW87 pad 2: (no net) -> Net-(D87-Pad2)
- SW88 pad 1: (no net) -> col14
- SW88 pad 2: (no net) -> Net-(D88-Pad2)
- SW89 pad 1: (no net) -> col14
- SW89 pad 2: (no net) -> Net-(D89-Pad2)
- SW9 pad 1: (no net) -> col01
- SW9 pad 2: (no net) -> Net-(D9-Pad2)
- SW90 pad 1: (no net) -> col14
- SW90 pad 2: (no net) -> Net-(D90-Pad2)
- SW91 pad 1: (no net) -> software_reset
- SW91 pad 2: (no net) -> GND
- SW92 pad 1: (no net) -> hardware_reset
- SW92 pad 2: (no net) -> GND
- SW93 pad 1: (no net) -> Net-(SW93-Pad1)
- SW93 pad 2: (no net) -> Net-(J2-Pad38)
- SW93 pad 3: (no net) -> VCC
- U1 pad 1: (no net) -> Net-(U1-Pad1)
- U1 pad 10: (no net) -> SCL
- U1 pad 11: (no net) -> RCK
- U1 pad 12: (no net) -> OE
- U1 pad 13: (no net) -> row05
- U1 pad 14: (no net) -> row04
- U1 pad 15: (no net) -> row03
- U1 pad 16: (no net) -> row02
- U1 pad 17: (no net) -> row01
- U1 pad 18: (no net) -> row00
- U1 pad 19: (no net) -> Net-(U1-Pad19)
- U1 pad 2: (no net) -> Net-(U1-Pad2)
- U1 pad 20: (no net) -> Net-(U1-Pad20)
- U1 pad 21: (no net) -> VCC
- U1 pad 22: (no net) -> hardware_reset
- U1 pad 23: (no net) -> GND
- U1 pad 24: (no net) -> Net-(U1-Pad24)
- U1 pad 3: (no net) -> GND
- U1 pad 4: (no net) -> GND
- U1 pad 5: (no net) -> Net-(U1-Pad5)
- U1 pad 6: (no net) -> Net-(U1-Pad6)
- U1 pad 7: (no net) -> software_reset
- U1 pad 8: (no net) -> SER
- U1 pad 9: (no net) -> SCK
- U2 pad 1: (no net) -> Net-(U2-Pad1)
- U2 pad 10: (no net) -> SCL
- U2 pad 11: (no net) -> RCK
- U2 pad 12: (no net) -> OE
- U2 pad 13: (no net) -> row05
- U2 pad 14: (no net) -> row04
- U2 pad 15: (no net) -> row03
- U2 pad 16: (no net) -> row02
- U2 pad 17: (no net) -> row01
- U2 pad 18: (no net) -> row00
- U2 pad 19: (no net) -> Net-(U2-Pad19)
- U2 pad 2: (no net) -> Net-(U2-Pad2)
- U2 pad 20: (no net) -> Net-(U2-Pad20)
- U2 pad 21: (no net) -> VCC
- U2 pad 22: (no net) -> hardware_reset
- U2 pad 23: (no net) -> GND
- U2 pad 24: (no net) -> Net-(U2-Pad24)
- U2 pad 3: (no net) -> GND
- U2 pad 4: (no net) -> GND
- U2 pad 5: (no net) -> Net-(U2-Pad5)
- U2 pad 6: (no net) -> Net-(U2-Pad6)
- U2 pad 7: (no net) -> software_reset
- U2 pad 8: (no net) -> SER
- U2 pad 9: (no net) -> SCK
- U3 pad 1: (no net) -> col01
- U3 pad 10: (no net) -> SCL
- U3 pad 11: (no net) -> SCK
- U3 pad 12: (no net) -> RCK
- U3 pad 13: (no net) -> OE
- U3 pad 14: (no net) -> SER
- U3 pad 15: (no net) -> col00
- U3 pad 16: (no net) -> VCC
- U3 pad 2: (no net) -> col02
- U3 pad 3: (no net) -> col03
- U3 pad 4: (no net) -> col04
- U3 pad 5: (no net) -> col05
- U3 pad 6: (no net) -> col06
- U3 pad 7: (no net) -> col07
- U3 pad 8: (no net) -> GND
- U3 pad 9: (no net) -> QHSER
- U4 pad 1: (no net) -> col09
- U4 pad 10: (no net) -> SCL
- U4 pad 11: (no net) -> SCK
- U4 pad 12: (no net) -> RCK
- U4 pad 13: (no net) -> OE
- U4 pad 14: (no net) -> QHSER
- U4 pad 15: (no net) -> col08
- U4 pad 16: (no net) -> VCC
- U4 pad 2: (no net) -> col10
- U4 pad 3: (no net) -> col11
- U4 pad 4: (no net) -> col12
- U4 pad 5: (no net) -> col13
- U4 pad 6: (no net) -> col14
- U4 pad 7: (no net) -> Net-(U4-Pad7)
- U4 pad 8: (no net) -> GND
- U4 pad 9: (no net) -> Net-(U4-Pad9)
- U5 pad 1: (no net) -> col01
- U5 pad 10: (no net) -> SCL
- U5 pad 11: (no net) -> SCK
- U5 pad 12: (no net) -> RCK
- U5 pad 13: (no net) -> OE
- U5 pad 14: (no net) -> SER
- U5 pad 15: (no net) -> col00
- U5 pad 16: (no net) -> VCC
- U5 pad 2: (no net) -> col02
- U5 pad 3: (no net) -> col03
- U5 pad 4: (no net) -> col04
- U5 pad 5: (no net) -> col05
- U5 pad 6: (no net) -> col06
- U5 pad 7: (no net) -> col07
- U5 pad 8: (no net) -> GND
- U5 pad 9: (no net) -> QHSER'
- U6 pad 1: (no net) -> col09
- U6 pad 10: (no net) -> SCL
- U6 pad 11: (no net) -> SCK
- U6 pad 12: (no net) -> RCK
- U6 pad 13: (no net) -> OE
- U6 pad 14: (no net) -> QHSER'
- U6 pad 15: (no net) -> col08
- U6 pad 16: (no net) -> VCC
- U6 pad 2: (no net) -> col10
- U6 pad 3: (no net) -> col11
- U6 pad 4: (no net) -> col12
- U6 pad 5: (no net) -> col13
- U6 pad 6: (no net) -> col14
- U6 pad 7: (no net) -> Net-(U6-Pad7)
- U6 pad 8: (no net) -> GND
- U6 pad 9: (no net) -> Net-(U6-Pad9)
Routing:
- net (no net): track 11725.6 -> 3.66 mm, vias 448 -> 0
- net row03: track 0.00 -> 527.0 mm, vias 0 -> 1
- net row04: track 0.00 -> 521.0 mm, vias 0 -> 1
- net row02: track 0.00 -> 517.0 mm, vias 0 -> 2
- net row05: track 0.00 -> 515.0 mm
- net row01: track 0.00 -> 509.3 mm, vias 0 -> 4
- net col14: track 0.00 -> 489.3 mm, vias 0 -> 5
- net col13: track 0.00 -> 460.4 mm, vias 0 -> 6
- net col12: track 0.00 -> 456.5 mm, vias 0 -> 6
- net col11: track 0.00 -> 444.0 mm, vias 0 -> 6
- net row00: track 0.00 -> 438.8 mm
- net col10: track 0.00 -> 423.6 mm, vias 0 -> 6
- net col00: track 0.00 -> 345.6 mm, vias 0 -> 4
- net col09: track 0.00 -> 344.7 mm, vias 0 -> 7
- net col01: track 0.00 -> 338.8 mm, vias 0 -> 3
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- added copper zone on B.Cu, net GND
- added copper zone on F.Cu, net GND
- removed copper zone on B.Cu, net (none)
- removed copper zone on F.Cu, net (none)
